File: 02PCB_Design/01KiCad_Project/HalfBridgePowerStage.kicad_sch (KiCad schematic)
At the start: 24 parts, among them U5 LMG2100R044RARR, U6 INA240A1PW

Commit message: Layout progress
Parts:
- U5: footprint (none) -> footprints:RAR0016B-MFG
- U6: footprint (none) -> Package_SO:TSSOP-8_4.4x3mm_P0.65mm
- renumbered C17 to C18, C18 to C19, C19 to C20, C20 to C21, C21 to C22, C22 to C23, C23 to C24, C24 to C25, C25 to C26, C26 to C27, C27 to C28, C28 to C29, C29 to C30, C30 to C31, C31 to C32, R11 to R10, R12 to R11, R13 to R12, R14 to R13, R15 to R14, R16 to R15, R10 to R9

Commit message: Design 1.0 Finished
Parts:
- renumbered R12 to R10, R13 to R11, R14 to R12, R15 to R13, R9 to R7, R10 to R8, R11 to R9
Other:
- moved on the sheet: C30, C31, C32, R11, R12, R13, U6
