File: 02PCB_Design/01KiCad_Project/HalfBridgePowerStage.kicad_sch (KiCad schematic)
At the start: 24 parts, among them U5 LMG2100R044RARR, U6 INA240A1PW

Commit message: Changed Some Capacitor Sizes, Added Capacitors in Power Gen
Parts:
- C26: renamed from C20; footprint Capacitor_SMD:C_0805_2012Metric_Pad1.18x1.45mm_HandSolder -> Capacitor_SMD:C_0603_1608Metric_Pad1.08x0.95mm_HandSolder
- C27: renamed from C21; footprint Capacitor_SMD:C_0805_2012Metric_Pad1.18x1.45mm_HandSolder -> Capacitor_SMD:C_0603_1608Metric_Pad1.08x0.95mm_HandSolder
- C28: renamed from C22; footprint Capacitor_SMD:C_0805_2012Metric_Pad1.18x1.45mm_HandSolder -> Capacitor_SMD:C_0603_1608Metric_Pad1.08x0.95mm_HandSolder
- R10, R7: value 3R -> 10R
- renumbered C18 to C24, C19 to C25, C23 to C29, C24 to C30, C25 to C31, C26 to C32, C27 to C33, C28 to C34, C29 to C35, C30 to C36, C31 to C37, C32 to C38
Other:
- note added: "Referenz Pins Überprüfen"

Commit message: edited footprints
Parts:
- U5: footprint footprints:RAR0016B-MFG -> MyFootprintLib:RAR0016B-MFG

Commit message: relayout in progress
Parts:
- C25, C34, C35, C36, C38: value 0.1uF -> 100nF
- C32, C33: value 47p -> 47pF
- R11: value 3.3m -> 3m
- R8, R9: value 20 -> 20R
Changed lines of the file:
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@@
       (effects (font (size 1.27 1.27)) (justify left))
     )
-    (property "Value" "0.1uF" (at 124.46 50.8 0)
+    (property "Value" "100nF" (at 124.46 50.8 0)
       (effects (font (size 1.27 1.27)) (justify left))
     )
@@
       (effects (font (size 1.27 1.27)) (justify left))
     )
-    (property "Value" "0.1uF" (at 109.22 143.51 0)
+    (property "Value" "100nF" (at 109.22 143.51 0)
       (effects (font (size 1.27 1.27)) (justify left))
     )
@@
       (effects (font (size 1.27 1.27)))
     )
-    (property "Value" "3.3m" (at 66.04 123.19 90)
+    (property "Value" "3m" (at 66.04 123.19 90)
       (effects (font (size 1.27 1.27)))
     )
@@
       (effects (font (size 1.27 1.27)) (justify left))
     )
-    (property "Value" "0.1uF" (at 95.25 166.37 0)
+    (property "Value" "100nF" (at 95.25 166.37 0)
       (effects (font (size 1.27 1.27)) (justify left))
     )
@@
       (effects (font (size 1.27 1.27)) (justify left))
     )
-    (property "Value" "47p" (at 62.23 78.74 0)
+    (property "Value" "47pF" (at 62.23 78.74 0)
       (effects (font (size 1.27 1.27)) (justify left))
     )
@@
       (effects (font (size 1.27 1.27)) (justify left))
     )
-    (property "Value" "47p" (at 53.34 82.55 0)
+    (property "Value" "47pF" (at 53.34 82.55 0)
       (effects (font (size 1.27 1.27)) (justify left))
     )
@@
       (effects (font (size 1.27 1.27)))
     )
-    (property "Value" "20" (at 54.61 67.31 90)
+    (property "Value" "20R" (at 54.61 67.31 90)
       (effects (font (size 1.27 1.27)))
     )
@@
       (effects (font (size 1.27 1.27)) (justify left))
     )
-    (property "Value" "0.1uF" (at 144.78 82.55 0)
+    (property "Value" "100nF" (at 144.78 82.55 0)
       (effects (font (size 1.27 1.27)) (justify left))
     )
@@
       (effects (font (size 1.27 1.27)) (justify left))
     )
-    (property "Value" "0.1uF" (at 124.46 82.55 0)
+    (property "Value" "100nF" (at 124.46 82.55 0)
       (effects (font (size 1.27 1.27)) (justify left))
     )
@@
       (effects (font (size 1.27 1.27)))
     )
-    (property "Value" "20" (at 45.72 72.39 90)
-      (effects (font (size 1.27 1.27)))
-    )
+    (property "Value" "20R" (at 45.72 72.39 90)
+      (effects (font (size 1.27 1.27)))
+    )
