File: 02PCB_Design/01KiCad_Project/NucleoMorpho.kicad_sch (KiCad schematic)
At the start: 24 parts, among them U11 NUCLEO-G431RB

Commit message: Layout progress
Parts:
- removed R44, R45: R, Resistor_SMD:R_0603_1608Metric_Pad0.98x0.95mm_HandSolder, symbol Device:R
- U11: footprint (none) -> footprints:NucleoMorphoG431RB
- renumbered C62 to C63, C63 to C64, C64 to C65, C65 to C66, C66 to C67, C67 to C68, C68 to C69, R31 to R30, R32 to R31, R33 to R32, R34 to R33, R35 to R34, R36 to R35, R37 to R36, R38 to R37, R39 to R38, R40 to R39, R41 to R40, R42 to R41, R43 to R42, R46 to R45
Connections:
- net +3.3V: now also U11.R_7 (VREFP); no longer U11.CN10_7 (VREFP)
- net +5V: now also U11.L_6 (E5V); no longer U11.CN7_6 (E5V)
- net 3.3V_EN: now also U11.L_32 (PA4); no longer U11.CN7_32 (PA4)
- net ENC_CS: now also U11.R_34 (PC4); no longer U11.CN10_34 (PC4)
- net GND: now also U11.L_19 (GND), U11.L_20 (GND), U11.L_22 (GND), U11.L_8 (GND), U11.R_20 (GND), U11.R_9 (GND); no longer U11.CN10_20 (GND), U11.CN10_9 (GND), U11.CN7_19 (GND), U11.CN7_20 (GND), U11.CN7_22 (GND), U11.CN7_8 (GND)
- net GNDA: now also U11.R_32 (AGND); no longer U11.CN10_32 (AGND)
- net IMU_CS: now also U11.R_6 (PC5); no longer U11.CN10_6 (PC5)
- net IMU_INT1: now also U11.R_22 (PB2); no longer U11.CN10_22 (PB2)
- net PWM_HI_U: now also U11.R_23 (PA8); no longer U11.CN10_23 (PA8)
- net PWM_HI_V: now also U11.R_21 (PA9); no longer U11.CN10_21 (PA9)
- net PWM_HI_W: now also U11.L_35 (PC2); no longer U11.CN7_35 (PC2)
- net PWM_LI_U: now also U11.R_14 (PA11); no longer U11.CN10_14 (PA11)
- net PWM_LI_V: now also U11.R_12 (PA12); no longer U11.CN10_12 (PA12)
- net PWM_LI_W: now also U11.R_24 (PB1); no longer U11.CN10_24 (PB1)
- net SPI_MISO: now also U11.R_33 (PA10); no longer U11.CN10_33 (PA10)
- net at R40.1: now also U11.R_19 (PC7); no longer U11.CN10_19 (PC7)
- net at C65.1, R36.1: now also U11.L_36 (PC1/PB9); no longer U11.CN7_36 (PC1/PB9)
- net at C67.1, R34.2: now also U11.L_30 (PA1), U11.L_34 (PB0); no longer U11.CN7_30 (PA1), U11.CN7_34 (PB0)
- net at R45.2: now also U11.R_5 (PB9); no longer U11.CN10_5 (PB9)
- net at C64.1, R35.1: now also U11.L_38 (PC0/PA15); no longer U11.CN7_38 (PC0/PA15)
- net at R30.2: now also U11.R_30 (PB13); no longer U11.CN10_30 (PB13)
- net at R41.1: now also U11.R_17 (PB6); no longer U11.CN10_17 (PB6)
- net at R42.2: now also U11.R_3 (PB8); no longer U11.CN10_3 (PB8)
- net at R39.2: now also U11.R_4 (PC6); no longer U11.CN10_4 (PC6)
- net at R32.1: now also U11.R_26 (PB15); no longer U11.CN10_26 (PB15)
- net at C69.1, R38.2: now also U11.R_15 (PA7); no longer U11.CN10_15 (PA7)
- net at C68.1, R37.2: now also U11.R_13 (PA6); no longer U11.CN10_13 (PA6)
- net at C63.1, R31.1: now also U11.R_28 (PB14); no longer U11.CN10_28 (PB14)
- net at C66.1, R33.2: now also U11.L_28 (PA0); no longer U11.CN7_28 (PA0)
- new net: U11.L_10 (NC), U11.L_11 (NC), U11.L_26 (NC), U11.L_9 (NC), U11.R_10 (NC), U11.R_36 (NC), U11.R_38 (NC)

Commit message: Design 1.0 Finished
Parts:
- renumbered R30 to R28, R31 to R29, R32 to R30, R33 to R31, R34 to R32, R35 to R33, R36 to R34, R37 to R35, R38 to R36, R39 to R37, R40 to R38, R41 to R39, R42 to R40, R45 to R41
