File: 02PCB_Design/01KiCad_Project/PowerGen.kicad_sch (KiCad schematic)
At the start: 25 parts, among them J3 FCR7350R, J4 FCR7350R

Commit message: Layout progress
Parts:
- removed R5, R6: 0R, Resistor_SMD:R_0603_1608Metric_Pad0.98x0.95mm_HandSolder, symbol Device:R
- removed R9: 100k, Resistor_SMD:R_0603_1608Metric_Pad0.98x0.95mm_HandSolder, symbol Device:R
- added C15: 4.7uF, Capacitor_SMD:C_0805_2012Metric_Pad1.18x1.45mm_HandSolder, symbol Device:C
- C16: renamed from C15; value 47uF -> 4.7uF; footprint Capacitor_THT:CP_Radial_D8.0mm_P3.50mm -> Capacitor_SMD:C_0805_2012Metric_Pad1.18x1.45mm_HandSolder
- J3, J4: footprint (none) -> Connector:Banana_Jack_1Pin
- L1: footprint (none) -> Inductor_SMD:L_Wuerth_MAPI-4020
- NT1, NT2: footprint (none) -> NetTie:NetTie-2_SMD_Pad0.5mm
- U3: value ~ -> L6982; footprint (none) -> Package_SO:TSSOP-8_3x3mm_P0.65mm
- U4: value ~ -> AP2114D; footprint (none) -> Package_TO_SOT_SMD:TO-252-2
- renumbered C16 to C17
Connections:
- net +24V: now also J4.1 (P$1), U3.5 (EN/CLKIN), U3.7 (VIN); no longer J4.P$2 (P$1), U3. (VOUT/FB)
- net +3.3V: now also U4.2 (VOUT); no longer U4. (VOUT)
- net +5V: now also U3.4 (VOUT/FB), U4.3 (VIN), C15.1; no longer U3. (VOUT/FB), U4. (VOUT)
- net GNDA: now also U3.6 (AGND), U4.1 (GND), C15.2; no longer C7.2, U3. (VOUT/FB), U4. (VOUT)
- net GNDPWR: now also C7.2, J3.1 (P$1), U3.8 (PGND); no longer J3.P$2 (P$1)
- net at C4.1, L1.1: now also U3.1 (SW); no longer U3. (VOUT/FB)
- net at C4.2: now also U3.2 (BOOT); no longer U3. (VOUT/FB)
- net at C6.1: now also U3.3 (VCC); no longer U3. (VOUT/FB)
- removed net EN_3.3V: U4. (VOUT)
Other:
- moved on the sheet: NT2, U4

Commit message: Design 1.0 Finished
Parts:
- removed NT1, NT2: NetTie_2, NetTie:NetTie-2_SMD_Pad0.5mm, symbol Device:NetTie_2
- renumbered R7 to R5, R8 to R6
Connections:
- net GNDPWR is gone; now on net GNDA: C10.2, C11.2, C12.2, C13.2, C14.2, C7.2, C8.2, C9.2, J3.1 (P$1), J3.P$1, J3.P$3 (P$1), J3.P$4 (P$1), J3.P$5 (P$1), U3.8 (PGND)
Changed lines of the file:
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@@
   (junction (at 64.77 72.39) (diameter 0) (color 0 0 0 0)
   )
-  (junction (at 116.84 118.11) (diameter 0) (color 0 0 0 0)
-  )
-  (junction (at 99.06 118.11) (diameter 0) (color 0 0 0 0)
-  )
   (junction (at 85.09 72.39) (diameter 0) (color 0 0 0 0)
   )
@@
     (stroke (width 0) (type default))
   )
-  (wire (pts (xy 116.84 111.76) (xy 116.84 118.11))
+  (wire (pts (xy 116.84 111.76) (xy 116.84 123.19))
     (stroke (width 0) (type default))
   )
@@
     (stroke (width 0) (type default))
   )
-  (wire (pts (xy 99.06 118.11) (xy 105.41 118.11))
-    (stroke (width 0) (type default))
-  )
   (wire (pts (xy 128.27 62.23) (xy 135.89 62.23))
     (stroke (width 0) (type default))
@@
     (stroke (width 0) (type default))
   )
-  (wire (pts (xy 99.06 118.11) (xy 99.06 111.76))
-    (stroke (width 0) (type default))
-  )
   (wire (pts (xy 201.93 62.23) (xy 185.42 62.23))
     (stroke (width 0) (type default))
@@
     (stroke (width 0) (type default))
   )
-  (wire (pts (xy 116.84 118.11) (xy 116.84 123.19))
-    (stroke (width 0) (type default))
-  )
   (wire (pts (xy 49.53 129.54) (xy 68.58 129.54))
     (stroke (width 0) (type default))
@@
     (stroke (width 0) (type default))
   )
-  (wire (pts (xy 99.06 111.76) (xy 105.41 111.76))
+  (wire (pts (xy 99.06 111.76) (xy 116.84 111.76))
     (stroke (width 0) (type default))
   )
@@
     (stroke (width 0) (type default))
   )
-  (wire (pts (xy 110.49 111.76) (xy 116.84 111.76))
-    (stroke (width 0) (type default))
-  )
   (wire (pts (xy 43.18 72.39) (xy 54.61 72.39))
     (stroke (width 0) (type default))
@@
     (stroke (width 0) (type default))
   )
-  (wire (pts (xy 110.49 118.11) (xy 116.84 118.11))
-    (stroke (width 0) (type default))
-  )
-  (wire (pts (xy 99.06 121.92) (xy 99.06 118.11))
+  (wire (pts (xy 99.06 111.76) (xy 99.06 121.92))
     (stroke (width 0) (type default))
   )
@@
     )
   )
-  (symbol (lib_id "Device:NetTie_2") (at 107.95 111.76 0) (unit 1)
-    (in_bom no) (on_board yes) (dnp no)
-    (property "Reference" "NT1" (at 107.95 107.95 0)
-      (effects (font (size 1.27 1.27)) hide)
-    )
-    (property "Value" "NetTie_2" (at 107.95 110.49 0)
-      (effects (font (size 1.27 1.27)))
-    )
-    (property "Footprint" "NetTie:NetTie-2_SMD_Pad0.5mm" (at 107.95 111.76 0)
-      (effects (font (size 1.27 1.27)) hide)
-    )
-    (property "Datasheet" "~" (at 107.95 111.76 0)
-      (effects (font (size 1.27 1.27)) hide)
-    )
-    (pin "1")
-    (pin "2")
-    (instances
-      (project "Testplatine"
-        (path "/de27a806-41f8-462d-8678-2476d523bbd9/a9fc49c7-f356-4c2b-bdd5-d12f8bcc20f7/19fd2576-88a8-46b2-b66c-f5674461b1c9"
-          (reference "NT1") (unit 1)
-        )
-      )
-    )
-  )
   (symbol (lib_id "Device:C") (at 204.47 123.19 0) (unit 1)
     (in_bom yes) (on_board yes) (dnp no)
@@
   (symbol (lib_id "Device:R") (at 190.5 113.03 0) (unit 1)
     (in_bom yes) (on_board yes) (dnp no)
-    (property "Reference" "R7" (at 191.77 111.76 0)
+    (property "Reference" "R5" (at 191.77 111.76 0)
       (effects (font (size 1.27 1.27)) (justify left))
     )
@@
       (project "Testplatine"
         (path "/de27a806-41f8-462d-8678-2476d523bbd9/a9fc49c7-f356-4c2b-bdd5-d12f8bcc20f7/19fd2576-88a8-46b2-b66c-f5674461b1c9"
-          (reference "R7") (unit 1)
+          (reference "R5") (unit 1)
         )
       )
@@
   (symbol (lib_id "Device:R") (at 190.5 123.19 0) (unit 1)
     (in_bom yes) (on_board yes) (dnp no)
-    (property "Reference" "R8" (at 191.77 121.92 0)
+    (property "Reference" "R6" (at 191.77 121.92 0)
       (effects (font (size 1.27 1.27)) (justify left))
     )
@@
       (project "Testplatine"
         (path "/de27a806-41f8-462d-8678-2476d523bbd9/a9fc49c7-f356-4c2b-bdd5-d12f8bcc20f7/19fd2576-88a8-46b2-b66c-f5674461b1c9"
-          (reference "R8") (unit 1)
-        )
-      )
-    )
-  )
-  (symbol (lib_id "Device:NetTie_2") (at 107.95 118.11 0) (unit 1)
-    (in_bom no) (on_board yes) (dnp no)
-    (property "Reference" "NT2" (at 107.95 114.3 0)
-      (effects (font (size 1.27 1.27)))
-    )
-    (property "Value" "NetTie_2" (at 107.95 116.84 0)
-      (effects (font (size 1.27 1.27)))
-    )
-    (property "Footprint" "NetTie:NetTie-2_SMD_Pad0.5mm" (at 107.95 118.11 0)
-      (effects (font (size 1.27 1.27)) hide)
-    )
-    (property "Datasheet" "~" (at 107.95 118.11 0)
-      (effects (font (size 1.27 1.27)) hide)
-    )
-    (pin "1")
-    (pin "2")
-    (instances
-      (project "Testplatine"
-        (path "/de27a806-41f8-462d-8678-2476d523bbd9/a9fc49c7-f356-4c2b-bdd5-d12f8bcc20f7/19fd2576-88a8-46b2-b66c-f5674461b1c9"
-          (reference "NT2") (unit 1)
-        )
-      )
+          (reference "R6") (unit 1)
+        )
+      )
