File: 02PCB_Design/01KiCad_Project/Testplatine.kicad_pcb (KiCad board)
At the start: 4 copper layers, 217.9 x 112.1 mm, 143 parts, among them J2 Screw_Terminal_01x03, J3 FCR7350R, J4 FCR7350R, J5 DE9_Receptacle_MountingHoles, J6 MTSW-104-22-L-D-265-RA, J7 Conn_01x06_Pin, J8 RJ45-8N-B, U1 AS5047P-ATSM, U10 INA240A1PW, U11 NUCLEO-G431RB, U12 MCP2562FD, U2 ISM330BXTR, U3 L6982, U4 AP2114D, U5 LMG2100R044RARR, U6 INA240A1PW, U7 LMG2100R044RARR, U8 INA240A1PW, U9 LMG2100R044RARR

Commit message: Added Filters + CAN
Parts:
- C76, C77, R38, R42, U12: moved to B.Cu
- R28, R29, R31, R33, R34, R35, R36, R37: moved to F.Cu
- moved C45 192.4 mm to (93.4, 133.3), turned to 180 degrees
- moved C43 192.2 mm to (93.6, 131.4), turned to 180 degrees
- moved C48 188.9 mm to (94.3, 121.4), turned to 90 degrees
- moved C49 186.5 mm to (95.9, 125.1)
- moved C50 186.5 mm to (98.4, 124.2)
- moved R17 186.5 mm to (98.4, 126.0)
- moved C42 185.9 mm to (98.0, 129.4), turned to 0 degrees
- moved U8 185.9 mm to (75.1, 122.7)
- moved C40 185.9 mm to (89.4, 122.3)
- moved C51 185.9 mm to (77.2, 118.0)
- moved C52 185.9 mm to (67.0, 119.0)
- moved C53 185.9 mm to (73.8, 118.0)
- moved R14 185.9 mm to (91.0, 122.3)
- moved R18 185.9 mm to (75.1, 128.7)
- moved R19 185.9 mm to (68.8, 122.5)
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Routing:
- net /escSheet/Bus_Connectors/O_ENC_A: track 0.00 -> 40.7 mm
- net /escSheet/Bus_Connectors/O_ENC_I: track 0.00 -> 27.9 mm
- net /escSheet/Bus_Connectors/O_ENC_B: track 0.00 -> 27.8 mm
- net GNDA: track 78.4 -> 100.0 mm, vias 100 -> 145
- net /escSheet/Bus_Connectors/FDCAN_TX: track 0.00 -> 13.6 mm
- net Net-(U11A-PA1): track 0.00 -> 11.4 mm
- net /escSheet/Bus_Connectors/FDCAN_RX: track 0.00 -> 9.57 mm
- net Net-(U12-CANH): track 0.00 -> 9.01 mm
- net Net-(U12-CANL): track 0.00 -> 8.90 mm
- net Net-(U11A-PB8): track 0.00 -> 7.55 mm
- net Net-(U11A-PA7): track 0.00 -> 5.99 mm
- net Net-(U11A-PC0/PA15): track 0.00 -> 5.70 mm
- net Net-(U11A-PC1/PB9): track 0.00 -> 5.68 mm
- net Net-(U11A-PB14): track 0.00 -> 5.67 mm
- net Net-(U11A-PA6): track 0.00 -> 5.57 mm
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- added copper zone on B.Cu, net +3.3V
Other:
- board text added: "Kondensator Näher an GNDA (Pin4)?"

Commit message: main 5V supply
Parts:
- C69, C74, C75, R28, R29, R30, R35, R36: moved to B.Cu
- moved C21 35.6 mm to (26.9, 64.8), turned to 90 degrees
- moved C22 35.0 mm to (28.8, 64.6), turned to 90 degrees
- moved C20 29.8 mm to (19.6, 74.6), turned to 180 degrees
- moved U4 29.7 mm to (25.1, 70.2), turned to 0 degrees
- moved C19 28.3 mm to (19.5, 76.5), turned to 180 degrees
- moved J3 26.4 mm to (98.8, 48.8), turned to 0 degrees
- moved C7 25.9 mm to (67.7, 68.7)
- moved U3 25.8 mm to (71.6, 67.1)
- moved C10 25.8 mm to (77.2, 63.2)
- moved L1 25.8 mm to (76.9, 67.1)
- moved C11 25.8 mm to (79.7, 62.4)
- moved C8 25.8 mm to (71.7, 64.4)
- moved C9 25.8 mm to (75.6, 63.2)
- moved C4 25.8 mm to (73.4, 70.0)
- moved C6 24.6 mm to (67.4, 64.8), turned to -90 degrees
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Routing:
- net /escSheet/HalfBridgePowerStage3/PWM_LI: track 0.00 -> 90.4 mm, vias 0 -> 2
- net /escSheet/HalfBridgePowerStage1/PWM_LI: track 0.00 -> 87.7 mm, vias 0 -> 2
- net /escSheet/HalfBridgePowerStage2/PWM_LI: track 0.00 -> 82.9 mm
- net /escSheet/HalfBridgePowerStage3/PWM_HI: track 0.00 -> 70.6 mm
- net /escSheet/HalfBridgePowerStage2/PWM_HI: track 0.00 -> 70.1 mm, vias 0 -> 1
- net /escSheet/HalfBridgePowerStage1/PWM_HI: track 0.00 -> 68.5 mm, vias 0 -> 1
- net /escSheet/Bus_Connectors/SPI_MOSI: track 0.00 -> 32.5 mm
- net /escSheet/Bus_Connectors/SPI_SCLK: track 0.00 -> 27.9 mm
- net Net-(U11A-PA7): track 5.99 -> 0.00 mm
- net Net-(U11A-PA6): track 5.57 -> 0.14 mm
- net +5V: track 3.73 -> 8.47 mm, vias 1 -> 13
- net Net-(U11A-PB15): track 4.00 -> 2.13 mm
- net Net-(U11A-PB13): track 3.90 -> 2.06 mm
- net Net-(U11A-PB14): track 5.67 -> 4.22 mm
- net GNDA: track 100.0 -> 98.6 mm, vias 145 -> 146
- added copper zone on In2.Cu, net +5V
Other:
- board text removed: "Kondensator Näher an GNDA (Pin4)?"

Commit message: Added Signal Lines
Parts:
- C69, R29: moved to F.Cu
- C70, C71, C73, R32, R33, R34: moved to B.Cu
- moved C23 13.0 mm to (131.7, 45.6)
- moved R5 13.0 mm to (130.2, 49.0)
- moved R6 13.0 mm to (130.2, 45.6)
- moved C69 3.61 mm to (152.1, 116.2), turned to 180 degrees
- moved C73 2.62 mm to (149.2, 52.6)
- moved R32 2.56 mm to (150.8, 52.6)
- moved C71 2.05 mm to (144.8, 52.5)
- moved R34 2.05 mm to (143.2, 52.5)
- moved R33 2.04 mm to (140.6, 52.6)
- moved C70 2.04 mm to (138.9, 52.6)
- moved R29 1.40 mm to (152.0, 114.6), turned to 180 degrees
Connections:
- C71 pad 1: Net-(U11A-PC1/PB9) -> /escSheet/NucleoMorpho/Current_Comp
- R29 pad 2: /escSheet/HalfBridgePowerStage1/V_PHASE -> /escSheet/HalfBridgePowerStage2/V_PHASE
- R32 pad 1: /escSheet/HalfBridgePowerStage1/I_PHASE -> /escSheet/HalfBridgePowerStage1/V_PHASE
- R33 pad 2: /escSheet/HalfBridgePowerStage2/V_PHASE -> /escSheet/HalfBridgePowerStage3/V_PHASE
- R34 pad 1: Net-(U11A-PC1/PB9) -> /escSheet/NucleoMorpho/Current_Comp
- R34 pad 2: /escSheet/HalfBridgePowerStage3/V_PHASE -> /escSheet/HalfBridgePowerStage3/I_PHASE
- R35 pad 1: /escSheet/HalfBridgePowerStage2/I_PHASE -> /escSheet/HalfBridgePowerStage1/I_PHASE
- R36 pad 1: /escSheet/HalfBridgePowerStage3/I_PHASE -> /escSheet/HalfBridgePowerStage2/I_PHASE
- U11 pad L_34: Net-(U11A-PA1) -> /escSheet/NucleoMorpho/Current_Comp
- U11 pad L_36: Net-(U11A-PC1/PB9) -> /escSheet/NucleoMorpho/Current_Comp
Routing:
- net /escSheet/HalfBridgePowerStage1/V_PHASE: track 3.40 -> 119.3 mm
- net /escSheet/HalfBridgePowerStage2/I_PHASE: track 0.00 -> 109.5 mm, vias 0 -> 1
- net /escSheet/HalfBridgePowerStage1/I_PHASE: track 0.00 -> 104.1 mm, vias 0 -> 1
- net /escSheet/HalfBridgePowerStage2/V_PHASE: track 3.40 -> 93.1 mm, vias 0 -> 1
- net /escSheet/HalfBridgePowerStage3/V_PHASE: track 3.40 -> 92.1 mm
- net /escSheet/HalfBridgePowerStage3/I_PHASE: track 0.00 -> 88.3 mm, vias 0 -> 1
- net Net-(U11A-PA1): track 11.4 -> 3.72 mm
- net /escSheet/NucleoMorpho/Current_Comp: track 0.00 -> 6.67 mm
- net Net-(U11A-PC1/PB9): track 5.68 -> 0.00 mm
- net Net-(U11A-PA0): track 5.56 -> 0.10 mm
- net Net-(U11A-PB14): track 4.22 -> 6.78 mm
- net Net-(U11A-PC0/PA15): track 5.70 -> 3.83 mm

Commit message: All Signals Connected, Ethernet Cable
Parts:
- removed J8: RJ45-8N-B, RJ45-8N-B:TE_RJ45-8N-B
- added J1: RJ45-8N-B, RJ45-8N-B:TE_RJ45-8N-B, F.Cu at (229.8, 96.5)
- C19, C20, C21, C22, C23, C72, R31, R5, R6, U4: moved to B.Cu
- J6: value MTSW-104-22-L-D-265-RA -> RJ45-8N-B; footprint Connector_PinHeader_2.54mm:PinHeader_2x04_P2.54mm_Horizontal -> RJ45-8N-B:TE_RJ45-8N-B
- moved C22 31.1 mm to (57.4, 76.8), turned to -90 degrees
- moved C21 31.0 mm to (55.5, 76.6), turned to -90 degrees
- moved C19 30.9 mm to (48.1, 65.0)
- moved C20 29.7 mm to (48.3, 66.9)
- moved U4 28.7 mm to (53.7, 71.3)
- moved C72 11.8 mm to (151.2, 43.4), turned to 180 degrees
- moved R31 9.80 mm to (151.1, 45.1), turned to 0 degrees
- moved J6 5.32 mm to (126.9, 132.4), turned to 0 degrees
- moved R5 2.82 mm to (127.7, 47.6)
- moved R6 2.82 mm to (127.7, 44.2)
- moved C23 2.82 mm to (129.3, 44.2)
- moved C75 0.75 mm to (166.9, 105.1)
- moved R36 0.75 mm to (168.6, 105.1)
Connections:
- J6 pad 1: /escSheet/Bus_Connectors/SPI_SCLK -> +3.3V
- J6 pad 2: /escSheet/Bus_Connectors/SPI_MOSI -> unconnected-(J6-Pad2)
- J6 pad 3: /escSheet/Bus_Connectors/ENC_CS -> /escSheet/Bus_Connectors/IMU_INT1
- J6 pad 4: /escSheet/Bus_Connectors/IMU_CS -> /escSheet/Bus_Connectors/SPI_MISO
- J6 pad 5: /escSheet/Bus_Connectors/SPI_MISO -> /escSheet/Bus_Connectors/IMU_CS
- J6 pad 6: +3.3V -> /escSheet/Bus_Connectors/ENC_CS
- J6 pad 7: GNDA -> /escSheet/Bus_Connectors/SPI_MOSI
- J6 pad 8: /escSheet/Bus_Connectors/IMU_INT1 -> /escSheet/Bus_Connectors/SPI_SCLK
Routing:
- net +3.3V: track 19.9 -> 106.6 mm
- net /escSheet/Bus_Connectors/IMU_CS: track 0.00 -> 64.9 mm, vias 0 -> 2
- net /escSheet/Bus_Connectors/IMU_INT1: track 0.00 -> 43.8 mm, vias 0 -> 1
- net /escSheet/Bus_Connectors/SPI_MISO: track 0.00 -> 26.9 mm, vias 0 -> 1
- net /escSheet/NucleoMorpho/VOLTAGE_BUS: track 0.00 -> 24.0 mm
- net /escSheet/Bus_Connectors/ENC_CS: track 0.00 -> 23.7 mm, vias 0 -> 1
- net GNDA: track 98.6 -> 106.8 mm, vias 146 -> 151
- net Net-(U11A-PA0): track 0.10 -> 6.81 mm
- net /SensorSheet/SPI_MISO: track 33.8 -> 38.9 mm
- net /SensorSheet/SPI_MOSI: track 37.7 -> 32.6 mm, vias 1 -> 2
- net +5V: track 8.47 -> 3.73 mm
- net /SensorSheet/ENC_CS: track 18.0 -> 13.9 mm, vias 2 -> 1
- net Net-(U11A-PA6): track 0.14 -> 3.83 mm
- net Net-(U11A-PA7): track 0.00 -> 3.61 mm
- net +24V: track 0.00 -> 3.53 mm, vias 45 -> 46
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- added copper zone on B.Cu, net +5V
- added copper zone on B.Cu, net GNDA
- removed copper zone on F.Cu, net +3.3V
Other:
- board text removed: "Falsch Herum?"
