File: 02PCB_Design/01KiCad_Project/escSheet.kicad_sch (KiCad schematic)
At the start: 1 part, among them J2 Screw_Terminal_01x03

Commit message: Via stitching and edited footprints
Parts:
- added H4, H5, H6, H7: MountingHole, MountingHole:MountingHole_4.3mm_M4_Pad_Via, symbol Mechanical:MountingHole
Changed lines of the file:
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@@
     (effects (font (size 2 2)) (justify left top))
+  )
+  (symbol (lib_id "Mechanical:MountingHole") (at 24.13 167.64 0) (unit 1)
+    (in_bom yes) (on_board yes) (dnp no) (fields_autoplaced)
+    (property "Reference" "H4" (at 26.67 166.37 0)
+      (effects (font (size 1.27 1.27)) (justify left))
+    )
+    (property "Value" "MountingHole" (at 26.67 168.91 0)
+      (effects (font (size 1.27 1.27)) (justify left))
+    )
+    (property "Footprint" "MountingHole:MountingHole_4.3mm_M4_Pad_Via" (at 24.13 167.64 0)
+      (effects (font (size 1.27 1.27)) hide)
+    )
+    (property "Datasheet" "~" (at 24.13 167.64 0)
+      (effects (font (size 1.27 1.27)) hide)
+    )
+    (instances
+      (project "Testplatine"
+        (path "/de27a806-41f8-462d-8678-2476d523bbd9/a9fc49c7-f356-4c2b-bdd5-d12f8bcc20f7"
+          (reference "H4") (unit 1)
+        )
+      )
+    )
+  )
+  (symbol (lib_id "Mechanical:MountingHole") (at 24.13 172.72 0) (unit 1)
+    (in_bom yes) (on_board yes) (dnp no) (fields_autoplaced)
+    (property "Reference" "H5" (at 26.67 171.45 0)
+      (effects (font (size 1.27 1.27)) (justify left))
+    )
+    (property "Value" "MountingHole" (at 26.67 173.99 0)
+      (effects (font (size 1.27 1.27)) (justify left))
+    )
+    (property "Footprint" "MountingHole:MountingHole_4.3mm_M4_Pad_Via" (at 24.13 172.72 0)
+      (effects (font (size 1.27 1.27)) hide)
+    )
+    (property "Datasheet" "~" (at 24.13 172.72 0)
+      (effects (font (size 1.27 1.27)) hide)
+    )
+    (instances
+      (project "Testplatine"
+        (path "/de27a806-41f8-462d-8678-2476d523bbd9/a9fc49c7-f356-4c2b-bdd5-d12f8bcc20f7"
+          (reference "H5") (unit 1)
+        )
+      )
+    )
   )
   (symbol (lib_id "Connector:Screw_Terminal_01x03") (at 251.46 106.68 0) (unit 1)
@@
         )
       )
+    )
+  )
+  (symbol (lib_id "Mechanical:MountingHole") (at 24.13 182.88 0) (unit 1)
+    (in_bom yes) (on_board yes) (dnp no) (fields_autoplaced)
+    (property "Reference" "H7" (at 26.67 181.61 0)
+      (effects (font (size 1.27 1.27)) (justify left))
+    )
+    (property "Value" "MountingHole" (at 26.67 184.15 0)
+      (effects (font (size 1.27 1.27)) (justify left))
+    )
+    (property "Footprint" "MountingHole:MountingHole_4.3mm_M4_Pad_Via" (at 24.13 182.88 0)
+      (effects (font (size 1.27 1.27)) hide)
+    )
+    (property "Datasheet" "~" (at 24.13 182.88 0)
+      (effects (font (size 1.27 1.27)) hide)
+    )
+    (instances
+      (project "Testplatine"
+        (path "/de27a806-41f8-462d-8678-2476d523bbd9/a9fc49c7-f356-4c2b-bdd5-d12f8bcc20f7"
+          (reference "H7") (unit 1)
+        )
+      )
+    )
+  )
+  (symbol (lib_id "Mechanical:MountingHole") (at 24.13 177.8 0) (unit 1)
+    (in_bom yes) (on_board yes) (dnp no) (fields_autoplaced)
+    (property "Reference" "H6" (at 26.67 176.53 0)
+      (effects (font (size 1.27 1.27)) (justify left))
+    )
+    (property "Value" "MountingHole" (at 26.67 179.07 0)
+      (effects (font (size 1.27 1.27)) (justify left))
+    )
+    (property "Footprint" "MountingHole:MountingHole_4.3mm_M4_Pad_Via" (at 24.13 177.8 0)
+      (effects (font (size 1.27 1.27)) hide)
+    )
+    (property "Datasheet" "~" (at 24.13 177.8 0)
+      (effects (font (size 1.27 1.27)) hide)
+    )
+    (instances
+      (project "Testplatine"
+        (path "/de27a806-41f8-462d-8678-2476d523bbd9/a9fc49c7-f356-4c2b-bdd5-d12f8bcc20f7"
+          (reference "H6") (unit 1)
+        )
+      )

Commit message: Edited some connectors
Parts:
- removed H4: MountingHole, MountingHole:MountingHole_4.3mm_M4_Pad_Via, symbol Mechanical:MountingHole
- H5, H6, H7: symbol Mechanical:MountingHole -> Mechanical:MountingHole_Pad
Connections:
- new net GNDA: H5.1, H6.1, H7.1
Changed lines of the file:
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@@
 (kicad_sch (version 20230121) (generator eeschema)
   (paper "A4")
+  (junction (at 35.56 176.53) (diameter 0) (color 0 0 0 0)
+  )
+  (junction (at 35.56 171.45) (diameter 0) (color 0 0 0 0)
+  )
   (wire (pts (xy 134.62 72.39) (xy 171.45 72.39))
     (stroke (width 0) (type default))
   )
+  (wire (pts (xy 35.56 171.45) (xy 35.56 176.53))
+    (stroke (width 0) (type default))
+  )
   (wire (pts (xy 134.62 64.77) (xy 171.45 64.77))
     (stroke (width 0) (type default))
@@
     (stroke (width 0) (type default))
   )
+  (wire (pts (xy 35.56 166.37) (xy 35.56 171.45))
+    (stroke (width 0) (type default))
+  )
   (wire (pts (xy 228.6 106.68) (xy 246.38 106.68))
     (stroke (width 0) (type default))
@@
     (stroke (width 0) (type default))
   )
+  (wire (pts (xy 35.56 186.69) (xy 49.53 186.69))
+    (stroke (width 0) (type default))
+  )
   (wire (pts (xy 134.62 102.87) (xy 171.45 102.87))
     (stroke (width 0) (type default))
@@
     (stroke (width 0) (type default))
   )
+  (wire (pts (xy 49.53 186.69) (xy 49.53 187.96))
+    (stroke (width 0) (type default))
+  )
   (wire (pts (xy 82.55 152.4) (xy 95.25 152.4))
+    (stroke (width 0) (type default))
+  )
+  (wire (pts (xy 35.56 176.53) (xy 35.56 186.69))
     (stroke (width 0) (type default))
   )
@@
     (effects (font (size 2 2)) (justify left top))
   )
-  (symbol (lib_id "Mechanical:MountingHole") (at 24.13 167.64 0) (unit 1)
-    (in_bom yes) (on_board yes) (dnp no) (fields_autoplaced)
-    (property "Reference" "H4" (at 26.67 166.37 0)
-      (effects (font (size 1.27 1.27)) (justify left))
-    )
-    (property "Value" "MountingHole" (at 26.67 168.91 0)
-      (effects (font (size 1.27 1.27)) (justify left))
-    )
-    (property "Footprint" "MountingHole:MountingHole_4.3mm_M4_Pad_Via" (at 24.13 167.64 0)
-      (effects (font (size 1.27 1.27)) hide)
-    )
-    (property "Datasheet" "~" (at 24.13 167.64 0)
-      (effects (font (size 1.27 1.27)) hide)
-    )
-    (instances
-      (project "Testplatine"
-        (path "/de27a806-41f8-462d-8678-2476d523bbd9/a9fc49c7-f356-4c2b-bdd5-d12f8bcc20f7"
-          (reference "H4") (unit 1)
-        )
-      )
-    )
-  )
-  (symbol (lib_id "Mechanical:MountingHole") (at 24.13 172.72 0) (unit 1)
-    (in_bom yes) (on_board yes) (dnp no) (fields_autoplaced)
-    (property "Reference" "H5" (at 26.67 171.45 0)
-      (effects (font (size 1.27 1.27)) (justify left))
-    )
-    (property "Value" "MountingHole" (at 26.67 173.99 0)
-      (effects (font (size 1.27 1.27)) (justify left))
-    )
-    (property "Footprint" "MountingHole:MountingHole_4.3mm_M4_Pad_Via" (at 24.13 172.72 0)
-      (effects (font (size 1.27 1.27)) hide)
-    )
-    (property "Datasheet" "~" (at 24.13 172.72 0)
-      (effects (font (size 1.27 1.27)) hide)
-    )
+  (symbol (lib_id "power:GNDA") (at 49.53 187.96 0) (unit 1)
+    (in_bom yes) (on_board yes) (dnp no)
+    (property "Reference" "#PWR089" (at 49.53 194.31 0)
+      (effects (font (size 1.27 1.27)) hide)
+    )
+    (property "Value" "GNDA" (at 49.53 191.77 0)
+      (effects (font (size 1.27 1.27)))
+    )
+    (property "Footprint" "" (at 49.53 187.96 0)
+      (effects (font (size 1.27 1.27)) hide)
+    )
+    (property "Datasheet" "" (at 49.53 187.96 0)
+      (effects (font (size 1.27 1.27)) hide)
+    )
+    (pin "1")
+    (instances
+      (project "Testplatine"
+        (path "/de27a806-41f8-462d-8678-2476d523bbd9/a9fc49c7-f356-4c2b-bdd5-d12f8bcc20f7"
+          (reference "#PWR089") (unit 1)
+        )
+      )
+    )
+  )
+  (symbol (lib_id "Mechanical:MountingHole_Pad") (at 38.1 176.53 270) (unit 1)
+    (in_bom yes) (on_board yes) (dnp no) (fields_autoplaced)
+    (property "Reference" "H5" (at 41.91 175.26 90)
+      (effects (font (size 1.27 1.27)) (justify left))
+    )
+    (property "Value" "MountingHole" (at 41.91 177.8 90)
+      (effects (font (size 1.27 1.27)) (justify left))
+    )
+    (property "Footprint" "MountingHole:MountingHole_4.3mm_M4_Pad_Via" (at 38.1 176.53 0)
+      (effects (font (size 1.27 1.27)) hide)
+    )
+    (property "Datasheet" "~" (at 38.1 176.53 0)
+      (effects (font (size 1.27 1.27)) hide)
+    )
+    (pin "1")
     (instances
       (project "Testplatine"
@@
     )
   )
-  (symbol (lib_id "Mechanical:MountingHole") (at 24.13 182.88 0) (unit 1)
-    (in_bom yes) (on_board yes) (dnp no) (fields_autoplaced)
-    (property "Reference" "H7" (at 26.67 181.61 0)
-      (effects (font (size 1.27 1.27)) (justify left))
-    )
-    (property "Value" "MountingHole" (at 26.67 184.15 0)
-      (effects (font (size 1.27 1.27)) (justify left))
-    )
-    (property "Footprint" "MountingHole:MountingHole_4.3mm_M4_Pad_Via" (at 24.13 182.88 0)
-      (effects (font (size 1.27 1.27)) hide)
-    )
-    (property "Datasheet" "~" (at 24.13 182.88 0)
-      (effects (font (size 1.27 1.27)) hide)
-    )
+  (symbol (lib_id "Mechanical:MountingHole_Pad") (at 38.1 166.37 270) (unit 1)
+    (in_bom yes) (on_board yes) (dnp no) (fields_autoplaced)
+    (property "Reference" "H7" (at 41.91 165.1 90)
+      (effects (font (size 1.27 1.27)) (justify left))
+    )
+    (property "Value" "MountingHole" (at 41.91 167.64 90)
+      (effects (font (size 1.27 1.27)) (justify left))
+    )
+    (property "Footprint" "MountingHole:MountingHole_4.3mm_M4_Pad_Via" (at 38.1 166.37 0)
+      (effects (font (size 1.27 1.27)) hide)
+    )
+    (property "Datasheet" "~" (at 38.1 166.37 0)
+      (effects (font (size 1.27 1.27)) hide)
+    )
+    (pin "1")
     (instances
       (project "Testplatine"
@@
     )
   )
-  (symbol (lib_id "Mechanical:MountingHole") (at 24.13 177.8 0) (unit 1)
-    (in_bom yes) (on_board yes) (dnp no) (fields_autoplaced)
-    (property "Reference" "H6" (at 26.67 176.53 0)
-      (effects (font (size 1.27 1.27)) (justify left))
-    )
-    (property "Value" "MountingHole" (at 26.67 179.07 0)
-      (effects (font (size 1.27 1.27)) (justify left))
-    )
-    (property "Footprint" "MountingHole:MountingHole_4.3mm_M4_Pad_Via" (at 24.13 177.8 0)
-      (effects (font (size 1.27 1.27)) hide)
-    )
-    (property "Datasheet" "~" (at 24.13 177.8 0)
-      (effects (font (size 1.27 1.27)) hide)
-    )
-    (instances
-      (project "Testplatine"
+  (symbol (lib_id "Mechanical:MountingHole_Pad") (at 38.1 171.45 270) (unit 1)
+    (in_bom yes) (on_board yes) (dnp no) (fields_autoplaced)
+    (property "Reference" "H6" (at 41.91 170.18 90)
+      (effects (font (size 1.27 1.27)) (justify left))
+    )
+    (property "Value" "MountingHole" (at 41.91 172.72 90)
+      (effects (font (size 1.27 1.27)) (justify left))
+    )
+    (property "Footprint" "MountingHole:MountingHole_4.3mm_M4_Pad_Via" (at 38.1 171.45 0)
+      (effects (font (size 1.27 1.27)) hide)
+    )
+    (property "Datasheet" "~" (at 38.1 171.45 0)
+      (effects (font (size 1.27 1.27)) hide)
+    )
+    (pin "1")
+    (instances
+      (project "Testplatine"

Commit message: relayout in progress
Parts:
- J2: value Screw_Terminal_01x03 -> Wurth Elektronic 2365 Printklemme; footprint TerminalBlock_Phoenix:TerminalBlock_Phoenix_MKDS-3-3-5.08_1x03_P5.08mm_Horizontal -> MyFootprintLib:Wurth Elektronik 2365 Printklemme
Changed lines of the file:
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@@
-    (stroke (width 0) (type default))
-  )
-  (wire (pts (xy 35.56 186.69) (xy 49.53 186.69))
     (stroke (width 0) (type default))
   )
@@
     (stroke (width 0) (type default))
   )
-  (wire (pts (xy 49.53 186.69) (xy 49.53 187.96))
-    (stroke (width 0) (type default))
-  )
   (wire (pts (xy 82.55 152.4) (xy 95.25 152.4))
     (stroke (width 0) (type default))
   )
-  (wire (pts (xy 35.56 176.53) (xy 35.56 186.69))
+  (wire (pts (xy 35.56 176.53) (xy 35.56 179.07))
     (stroke (width 0) (type default))
   )
@@
     (effects (font (size 2 2)) (justify left top))
   )
-  (symbol (lib_id "power:GNDA") (at 49.53 187.96 0) (unit 1)
+  (symbol (lib_id "power:GNDA") (at 35.56 179.07 0) (unit 1)
     (in_bom yes) (on_board yes) (dnp no)
-    (property "Reference" "#PWR089" (at 49.53 194.31 0)
+    (property "Reference" "#PWR089" (at 35.56 185.42 0)
       (effects (font (size 1.27 1.27)) hide)
     )
-    (property "Value" "GNDA" (at 49.53 191.77 0)
+    (property "Value" "GNDA" (at 35.56 182.88 0)
       (effects (font (size 1.27 1.27)))
     )
-    (property "Footprint" "" (at 49.53 187.96 0)
+    (property "Footprint" "" (at 35.56 179.07 0)
       (effects (font (size 1.27 1.27)) hide)
     )
-    (property "Datasheet" "" (at 49.53 187.96 0)
+    (property "Datasheet" "" (at 35.56 179.07 0)
       (effects (font (size 1.27 1.27)) hide)
     )
@@
       (effects (font (size 1.27 1.27)) (justify left))
     )
-    (property "Value" "Screw_Terminal_01x03" (at 254 107.95 0)
+    (property "Value" "Wurth Elektronic 2365 Printklemme" (at 254 107.95 0)
       (effects (font (size 1.27 1.27)) (justify left))
     )
-    (property "Footprint" "TerminalBlock_Phoenix:TerminalBlock_Phoenix_MKDS-3-3-5.08_1x03_P5.08mm_Horizontal" (at 251.46 106.68 0)
+    (property "Footprint" "MyFootprintLib:Wurth Elektronik 2365 Printklemme" (at 251.46 106.68 0)
       (effects (font (size 1.27 1.27)) hide)
     )
